File: parts/CN/CN-BA3-03-03/CN-BA3-03-03-kicad/CN-BA3-03-03-kicad.kicad_pcb (KiCad board)
At the start: 2 copper layers, 42 x 42 mm, 6 parts, among them J1 Barrel_Jack_Switch, J2 Conn_01x02_Male, J3 Conn_01x02_Male, SW1 SW_DPDT_x2, SW2 SW_DPDT_x2

Commit message: A few new things and a few fixes.
Connections:
- J1 pad 2: Net-(J1-Pad2) -> GND
- J1 pad 3: GND -> Net-(J1-Pad3)
Routing:
- net GND: track 63.7 -> 58.4 mm
