File: parts/CN/CN-BA3-03-03/CN-BA3-03-03-kicad/CN-BA3-03-03-kicad.sch (KiCad schematic (older format))
At the start: 5 parts, among them J1 Barrel_Jack_Switch, J2 Conn_01x02_Male, J3 Conn_01x02_Male, SW1 SW_DPDT_x2, SW2 SW_DPDT_x2

Commit message: A few new things and a few fixes.
Connections:
- net GND: now also J1.2; no longer J1.3
Changed lines of the file:
@@
 $EndComp
-Wire Wire Line
-	7700 2400 7000 2400
-Wire Wire Line
-	7000 2400 7000 3400
 Wire Wire Line
 	7000 3400 1000 3400
@@
 Wire Wire Line
 	6000 2300 6200 2300
+Wire Wire Line
+	7700 2300 7000 2300
+Wire Wire Line
+	7000 2300 7000 3400
 $EndSCHEMATC
