File: parts/OBBB/OOBB-RASP-PICO-SHIELD-01/OOBB-RASP-PICO-SHIELD-01.kicad_pcb (KiCad board)
At the start: 2 copper layers, 21.6 x 67.3 mm, 18 parts, among them J1 MODULE-CONN-OOBB-BA-01, J10 MODULE-CONN-OOBB-BA-01, J11 Barrel_Jack_Switch, J12 MODULE-CONN-OOBB-BA-01, J13 MODULE-CONN-OOBB-BA-01, J14 MODULE-CONN-OOBB-BA-01, J2 MODULE-CONN-OOBB-BA-01, J3 MODULE-CONN-OOBB-BA-01, J4 HEAD-JSTSH-X-PI04-RS oom.lt/H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, J5 MODULE-CONN-OOBB-BA-01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

Commit message: PICO Shield breakout v001
Parts:
- added U2: MODULE-CONN-USB-MEGA-01, oomlout_OOMP_modules:MODULE-CONN-USB-MEGA-01, F.Cu at (140.0, 124.0)
Routing:
- net VIN: track 13.6 -> 33.0 mm
- net VOUT: track 51.6 -> 56.0 mm
- net Net-(U2-Pad3): track 0.00 -> 3.16 mm, vias 0 -> 1
- net Net-(U2-Pad2): track 0.00 -> 3.10 mm
- net GND: track 16.3 -> 17.1 mm
Other:
- board size 21.6 x 67.3 mm -> 21.6 x 71.9 mm
