File: parts/OBBB/OOBB-RASP-PICO-SHIELD-01/OOBB-RASP-PICO-SHIELD-01.kicad_sch (KiCad schematic)
At the start: 18 parts, among them J1 MODULE-CONN-OOBB-BA-01, J10 MODULE-CONN-OOBB-BA-01, J11 Barrel_Jack_Switch, J12 MODULE-CONN-OOBB-BA-01, J13 MODULE-CONN-OOBB-BA-01, J14 MODULE-CONN-OOBB-BA-01, J2 MODULE-CONN-OOBB-BA-01, J3 MODULE-CONN-OOBB-BA-01, J4 HEAD-JSTSH-X-PI04-RS oom.lt/H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, J5 MODULE-CONN-OOBB-BA-01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

Commit message: PICO Shield breakout v001
Parts:
- added U2: MODULE-CONN-USB-MEGA-01, oomlout_OOMP_modules:MODULE-CONN-USB-MEGA-01, symbol oomlout_OOMP_modules:MODULE-CONN-USB-MEGA-01
Connections:
- net GND: now also U2.5 (GND), U2.A1 (GND), U2.A12 (GND), U2.B1 (GND), U2.B12 (GND)
- net VIN: now also U2.1 (VBUS), U2.A4 (VBUS), U2.A9 (VBUS), U2.B4 (VBUS), U2.B9 (VBUS)
- new net: U2.2 (D-), U2.A7 (D-)
- new net: U2.3 (D+), U2.A6 (D+)
- new net: U2.6 (Shield), U2.S1 (SHIELD)
Other:
- note added: "MODULE-CONN-USB-MEGA-01 oom.lt/MCUMEGA"
Changed lines of the file:
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@@
   (junction (at 203.2 123.19) (diameter 0) (color 0 0 0 0)
   )
+  (junction (at 170.18 279.4) (diameter 0) (color 0 0 0 0)
+  )
   (junction (at 203.2 118.11) (diameter 0) (color 0 0 0 0)
   )
@@
   (junction (at 203.2 125.73) (diameter 0) (color 0 0 0 0)
   )
+  (junction (at 160.02 245.11) (diameter 0) (color 0 0 0 0)
+  )
   (junction (at 242.57 118.11) (diameter 0) (color 0 0 0 0)
   )
@@
     (stroke (width 0) (type default) (color 0 0 0 0))
   )
+  (wire (pts (xy 138.43 262.89) (xy 156.21 262.89))
+    (stroke (width 0) (type default) (color 0 0 0 0))
+  )
   (wire (pts (xy 213.36 105.41) (xy 219.71 105.41))
     (stroke (width 0) (type default) (color 0 0 0 0))
@@
     (stroke (width 0) (type default) (color 0 0 0 0))
   )
+  (wire (pts (xy 115.57 314.96) (xy 115.57 311.15))
+    (stroke (width 0) (type default) (color 0 0 0 0))
+  )
   (wire (pts (xy 143.51 93.98) (xy 143.51 106.68))
     (stroke (width 0) (type default) (color 0 0 0 0))
   )
+  (wire (pts (xy 156.21 250.19) (xy 162.56 250.19))
+    (stroke (width 0) (type default) (color 0 0 0 0))
+  )
   (wire (pts (xy 213.36 107.95) (xy 219.71 107.95))
     (stroke (width 0) (type default) (color 0 0 0 0))
@@
     (stroke (width 0) (type default) (color 0 0 0 0))
   )
+  (wire (pts (xy 138.43 257.81) (xy 152.4 257.81))
+    (stroke (width 0) (type default) (color 0 0 0 0))
+  )
   (wire (pts (xy 219.71 120.65) (xy 205.74 120.65))
     (stroke (width 0) (type default) (color 0 0 0 0))
@@
     (stroke (width 0) (type default) (color 0 0 0 0))
   )
+  (wire (pts (xy 160.02 245.11) (xy 162.56 245.11))
+    (stroke (width 0) (type default) (color 0 0 0 0))
+  )
   (wire (pts (xy 114.3 151.13) (xy 114.3 163.83))
     (stroke (width 0) (type default) (color 0 0 0 0))
@@
     (stroke (width 0) (type default) (color 0 0 0 0))
   )
+  (wire (pts (xy 170.18 260.35) (xy 170.18 279.4))
+    (stroke (width 0) (type default) (color 0 0 0 0))
+  )
   (wire (pts (xy 102.1902 30.8177) (xy 108.5402 30.8177))
     (stroke (width 0) (type default) (color 0 0 0 0))
@@
     (stroke (width 0) (type default) (color 0 0 0 0))
   )
+  (wire (pts (xy 160.02 238.76) (xy 160.02 245.11))
+    (stroke (width 0) (type default) (color 0 0 0 0))
+  )
   (wire (pts (xy 146.9199 68.7221) (xy 143.1099 68.7221))
     (stroke (width 0) (type default) (color 0 0 0 0))
@@
     (stroke (width 0) (type default) (color 0 0 0 0))
   )
+  (wire (pts (xy 170.18 279.4) (xy 170.18 311.15))
+    (stroke (width 0) (type default) (color 0 0 0 0))
+  )
   (wire (pts (xy 29.21 115.3675) (xy 29.21 109.0175))
     (stroke (width 0) (type default) (color 0 0 0 0))
@@
     (stroke (width 0) (type default) (color 0 0 0 0))
   )
+  (wire (pts (xy 172.72 314.96) (xy 115.57 314.96))
+    (stroke (width 0) (type default) (color 0 0 0 0))
+  )
   (wire (pts (xy 242.57 118.11) (xy 242.57 120.65))
     (stroke (width 0) (type default) (color 0 0 0 0))
@@
     (stroke (width 0) (type default) (color 0 0 0 0))
   )
+  (wire (pts (xy 152.4 252.73) (xy 152.4 257.81))
+    (stroke (width 0) (type default) (color 0 0 0 0))
+  )
   (wire (pts (xy 224.79 154.94) (xy 224.79 151.13))
     (stroke (width 0) (type default) (color 0 0 0 0))
@@
     (stroke (width 0) (type default) (color 0 0 0 0))
   )
+  (wire (pts (xy 138.43 245.11) (xy 160.02 245.11))
+    (stroke (width 0) (type default) (color 0 0 0 0))
+  )
   (wire (pts (xy 240.03 95.25) (xy 246.38 95.25))
     (stroke (width 0) (type default) (color 0 0 0 0))
@@
     (stroke (width 0) (type default) (color 0 0 0 0))
   )
+  (wire (pts (xy 162.56 279.4) (xy 170.18 279.4))
+    (stroke (width 0) (type default) (color 0 0 0 0))
+  )
   (wire (pts (xy 108.5402 68.8199) (xy 104.7302 68.8199))
     (stroke (width 0) (type default) (color 0 0 0 0))
   )
+  (wire (pts (xy 162.56 285.75) (xy 162.56 279.4))
+    (stroke (width 0) (type default) (color 0 0 0 0))
+  )
   (wire (pts (xy 213.36 69.85) (xy 219.71 69.85))
     (stroke (width 0) (type default) (color 0 0 0 0))
@@
     (stroke (width 0) (type default) (color 0 0 0 0))
   )
+  (wire (pts (xy 123.19 311.15) (xy 170.18 311.15))
+    (stroke (width 0) (type default) (color 0 0 0 0))
+  )
   (wire (pts (xy 33.02 33.02) (xy 29.21 33.02))
     (stroke (width 0) (type default) (color 0 0 0 0))
@@
     (stroke (width 0) (type default) (color 0 0 0 0))
   )
+  (wire (pts (xy 172.72 260.35) (xy 172.72 314.96))
+    (stroke (width 0) (type default) (color 0 0 0 0))
+  )
   (wire (pts (xy 213.36 80.01) (xy 219.71 80.01))
     (stroke (width 0) (type default) (color 0 0 0 0))
   )
   (wire (pts (xy 203.2 125.73) (xy 200.66 125.73))
+    (stroke (width 0) (type default) (color 0 0 0 0))
+  )
+  (wire (pts (xy 156.21 262.89) (xy 156.21 250.19))
+    (stroke (width 0) (type default) (color 0 0 0 0))
+  )
+  (wire (pts (xy 162.56 252.73) (xy 152.4 252.73))
     (stroke (width 0) (type default) (color 0 0 0 0))
   )
@@
   (text "MODULE-CONN-DCJP-21D-01\noom.lt/MCD2" (at 105.41 148.59 0)
     (effects (font (size 3 3)) (justify left bottom))
+  )
+  (text "MODULE-CONN-USB-MEGA-01\noom.lt/MCUMEGA" (at 105.41 227.33 0)
+    (effects (font (size 5 5)) (justify left bottom))
   )
   (global_label "GPIO13" (shape input) (at 140.97 104.14 180) (fields_autoplaced)
@@
     (property "Intersheet References" "${INTERSHEET_REFS}" (id 0) (at 204.0526 41.8306 0)
       (effects (font (size 1.27 1.27)) (justify right) hide)
+    )
+  )
+  (global_label "VIN" (shape input) (at 160.02 238.76 90) (fields_autoplaced)
+    (effects (font (size 1.27 1.27)) (justify left))
+    (property "Intersheet References" "${INTERSHEET_REFS}" (id 0) (at 160.0994 233.3231 90)
+      (effects (font (size 1.27 1.27)) (justify left) hide)
     )
   )
@@
     )
     (pin "1")
+  )
+  (symbol (lib_id "oomlout_OOMP_modules:MODULE-CONN-USB-MEGA-01") (at 147.32 240.03 0) (unit 1)
+    (in_bom yes) (on_board yes) (fields_autoplaced)
+    (property "Reference" "U2" (id 0) (at 144.145 237.49 0))
+    (property "Value" "MODULE-CONN-USB-MEGA-01" (id 1) (at 144.145 240.03 0))
+    (property "Footprint" "oomlout_OOMP_modules:MODULE-CONN-USB-MEGA-01" (id 2) (at 147.32 240.03 0)
+      (effects (font (size 1.27 1.27)) hide)
+    )
+    (property "Datasheet" "oom.lt/MCUMEGA" (id 3) (at 147.32 240.03 0)
+      (effects (font (size 1.27 1.27)) hide)
+    )
+    (pin "1")
+    (pin "2")
+    (pin "3")
+    (pin "4")
+    (pin "5")
+    (pin "6")
+    (pin "A1")
+    (pin "A10")
+    (pin "A11")
+    (pin "A12")
+    (pin "A2")
+    (pin "A3")
+    (pin "A4")
+    (pin "A5")
+    (pin "A6")
+    (pin "A7")
+    (pin "A8")
+    (pin "A9")
+    (pin "B1")
+    (pin "B10")
+    (pin "B11")
+    (pin "B12")
+    (pin "B2")
+    (pin "B3")
+    (pin "B4")
+    (pin "B5")
+    (pin "B8")
+    (pin "B9")
+    (pin "S1")
   )
   (symbol (lib_id "Connector:Barrel_Jack_Switch") (at 128.27 166.37 0) (mirror y) (unit 1)
@@
     (pin "1")
   )
+  (symbol (lib_id "power:GND") (at 162.56 285.75 0) (unit 1)
+    (in_bom yes) (on_board yes) (fields_autoplaced)
+    (property "Reference" "#PWR0133" (id 0) (at 162.56 292.1 0)
+      (effects (font (size 1.27 1.27)) hide)
+    )
+    (property "Value" "GND" (id 1) (at 162.56 290.7056 0))
+    (property "Footprint" "" (id 2) (at 162.56 285.75 0)
+      (effects (font (size 1.27 1.27)) hide)
+    )
+    (property "Datasheet" "" (id 3) (at 162.56 285.75 0)
+      (effects (font (size 1.27 1.27)) hide)
+    )
+    (pin "1")
+  )
   (symbol (lib_id "power:GND") (at 29.21 41.91 0) (unit 1)
     (in_bom yes) (on_board yes) (fields_autoplaced)
@@
       (reference "#PWR0132") (unit 1) (value "GND") (footprint "")
     )
+    (path "/e1fd0adf-607b-4e6c-bc90-3d8148f0706f"
+      (reference "#PWR0133") (unit 1) (value "GND") (footprint "")
+    )
     (path "/e6bfc9cf-8c20-4ff7-970d-c5fa6e3554af"
       (reference "C1") (unit 1) (value "CAPC-0603-X-NF100-V50") (footprint "Capacitor_SMD:C_0603_1608Metric")
@@
       (reference "U1") (unit 1) (value "LD1117S33TR_SOT223") (footprint "Package_TO_SOT_SMD:SOT-223-3_TabPin2")
     )
+    (path "/68e80d23-d146-4fb5-9a11-c28120ccf99d"
+      (reference "U2") (unit 1) (value "MODULE-CONN-USB-MEGA-01") (footprint "oomlout_OOMP_modules:MODULE-CONN-USB-MEGA-01")
+    )
     (path "/c2a4235f-dc13-4bf3-b9a7-ffaf790f0560"
